File: bldc_driver_hw/MCU.kicad_sch (KiCad schematic)
At the start: 0 parts

Commit message: wip
Parts:
- added C22, C27, C29, C33, C34, C56: 100nF, Capacitor_SMD:C_0603_1608Metric, symbol Device:C_Small
- added C23, C24, C28, C32, C37, C57: 10uF, Capacitor_SMD:C_0603_1608Metric, symbol Device:C_Small
- added C58, C59: 12pF, Capacitor_SMD:C_0603_1608Metric, symbol Device:C_Small
- added U9: STM32G474RETx, Package_QFP:LQFP-64_10x10mm_P0.5mm, symbol MCU_ST_STM32G4:STM32G474RETx
- added Y1: Crystal, symbol Device:Crystal
Connections:
- new net: C59.1, U9.4 (PC15), Y1.2
- new net: C32.1, C33.1, U9.64 (VDD)
- new net: C58.1, U9.3 (PC14), Y1.1
- new net: C22.1, C23.1, U9.16 (VDD)
- new net +3.3V: C24.1, C27.1, C28.1, C29.1, C34.1, C37.1, C56.1, C57.1, U9.1 (VBAT), U9.29 (VDDA), U9.32 (VDD), U9.48 (VDD)
- new net GND: C22.2, C23.2, C24.2, C27.2, C28.2, C29.2, C32.2, C33.2, C34.2, C37.2, C56.2, C57.2, C58.2, C59.2, U9.15 (VSS), U9.27 (VSSA), U9.31 (VSS), U9.47 (VSS), U9.63 (VSS)
- new net IN_H_U: U9.42 (PA8)
- new net IN_H_V: U9.40 (PC8)
- new net IN_H_W: U9.38 (PC6)
- new net IN_L_U: U9.43 (PA9)
- new net IN_L_V: U9.41 (PC9)
- new net IN_L_W: U9.39 (PC7)
- new net UART_MOTOR_RX: U9.60 (PB7)
- new net UART_MOTOR_TX: U9.59 (PB6)
- new net USB_D+: U9.46 (PA12)
- new net USB_D-: U9.49 (PA13)

Commit message: wip
Parts:
- added C63, C65, C66, C74: 100nF, Capacitor_SMD:C_0603_1608Metric, symbol Device:C_Small
- added C64: 10uF, Capacitor_SMD:C_0603_1608Metric, symbol Device:C_Small
- added C73: 1uF, Capacitor_SMD:C_0603_1608Metric, symbol Device:C_Small
- added JP1, JP2, JP3, JP4, JP5, JP6: SolderJumper_2_Open, Jumper:SolderJumper-2_P1.3mm_Open_RoundedPad1.0x1.5mm, symbol Jumper:SolderJumper_2_Open
- added L3: 600R / 100MHz, Resistor_SMD:R_1206_3216Metric, symbol Device:L
- added R64: 100k, Resistor_SMD:R_0805_2012Metric, symbol Device:R_Small
- added SW4: SW_Push, symbol Switch:SW_Push
- added U5: MCP1501-33xSN, Package_SO:SOIC-8_3.9x4.9mm_P1.27mm, symbol Reference_Voltage:MCP1501-33xSN
- C58, C59: value 12pF -> 18pF
- Y1: value Crystal -> 24MHz; footprint (none) -> Crystal:Crystal_HC49-U_Vertical
Connections:
- net +3.3V: now also JP6.1 (A), R64.2
- net GND: now also C63.2, C64.2, C65.2, C66.2, C73.2, C74.2, SW4.1, U5.2 (GND), U5.4 (GND), U5.5 (GND), U5.6 (GND)
- net IN_H_W: now also U9.39 (PC7); no longer U9.38 (PC6)
- net IN_L_W: now also U9.38 (PC6); no longer U9.39 (PC7)
- net UART_MOTOR_RX: now also JP4.2 (B); no longer U9.60 (PB7)
- net UART_MOTOR_TX: now also JP3.2 (B); no longer U9.59 (PB6)
- net USB_D-: now also U9.45 (PA11); no longer U9.49 (PA13)
- net at C59.1, Y1.2: now also U9.6 (PF1); no longer U9.4 (PC15)
- net at C58.1, Y1.1: now also U9.5 (PF0); no longer U9.3 (PC14)
- net CAN_EN: now reaches U9.2 (PC13)
- net ADC_CSA_V: now reaches U9.20 (PA6)
- net ADC_CSA_W: now reaches U9.21 (PA7)
- net ADC_CSA_U: now reaches U9.22 (PC4)
- net TEMP_SENSOR: now reaches U9.24 (PB0)
- net at U9.25 (PB1): now also U9.26 (PB2)
- net at U9.28 (VREF+): now also C66.1, C73.1, L3.2
- net HALL_EFF_W: now reaches U9.33 (PB11)
- net HALL_EFF_V: now reaches U9.35 (PB13)
- net HALL_EFF_U: now reaches U9.36 (PB14)
- net SCLK: now reaches U9.50 (PA14)
- net SWO: now reaches U9.56 (PB3)
- net at U9.61 (PB8): now also JP2.1 (A)
- net at U9.62 (PB9): now also JP1.1 (A)
- net at U9.7 (PG10): now also C63.1, R64.1, SW4.2
- new net: JP5.1 (A), U5.7 (OUT), U5.8 (FB)
- new net: C74.1, JP5.2 (B), JP6.2 (B), L3.1
- new net: JP3.1 (A), U9.59 (PB6)
- new net: JP4.1 (A), U9.60 (PB7)
- new net +5V: C64.1, C65.1, U5.1 (VDD), U5.3 (~{SHDN})
- new net CAN_RX: JP2.2 (B)
- new net CAN_TX: JP1.2 (B)
- new net SWDIO: U9.49 (PA13)
Other:
- note added: "OPAMP_FLR_IN"
- note added: "OPAMP_FLR_OUT"
- moved on the sheet: C22, C23, C24, C27, C28, C29, C32, C33, C34, C37, C56, C57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

Commit message: schematic finished pcb in progress
Parts:
- added R17: 47R, Resistor_SMD:R_0603_1608Metric, symbol Device:R_Small
- added TP10, TP11, TP12, TP13, TP14: TestPoint, TestPoint:TestPoint_Pad_D2.0mm, symbol Connector:TestPoint
- R16: renamed from R64; footprint Resistor_SMD:R_0805_2012Metric -> Resistor_SMD:R_0603_1608Metric
- SW1: renamed from SW4; footprint (none) -> Button_Switch_SMD:SW_SPST_TL3342
- renumbered C64 to C19, C65 to C20, C74 to C21, C63 to C22, C73 to C23, C66 to C24, C58 to C25, C59 to C26, C24 to C27, C27 to C29, C29 to C30, C23 to C31, C22 to C32, C32 to C34, C56 to C35, C57 to C36, C34 to C37, C37 to C38, JP1 to JP10, JP3 to JP7, JP4 to JP8, JP2 to JP9, L3 to L2, U9 to U6
Connections:
- net +3.3V: now also C31.1, C32.1, C33.1, C34.1, U6.16 (VDD), U6.64 (VDD)
- net at JP5.1 (A), U5.7 (OUT), U5.8 (FB): now also TP10.1
- net TEMP_SENS2: now reaches U6.13 (PA1)
- net at U6.14 (PA2): now also U6.17 (PA3), TP13.1
- net at U6.25 (PB1), U6.26 (PB2): now also TP14.1
- net at C23.1, C24.1, L2.2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: now also TP11.1
- net B_H_SENS_W: now reaches U6.34 (PB12)
- net H_BRIDGE_IRQ: now reaches U6.37 (PB15)
- net JTDI: now reaches U6.51 (PA15)
- net UART5_TX: now reaches U6.54 (PC12)
- net UART5_RX: now reaches U6.55 (PD2)
- net JTRST: now reaches U6.57 (PB4)
- net NRESET: now reaches C22.1, R16.1, SW1.2
- net NRESET: now also R17.2, TP12.1; no longer U6.7 (PG10)
- net HALL_EFF_U renamed B_H_SENS_U
- net HALL_EFF_V renamed B_H_SENS_V
- net HALL_EFF_W: no longer names the net of U6.33 (PB11)
- net SCLK renamed JTCK_SWCLK
- net SWDIO renamed JTMS_SWDIO
- net SWO renamed JTDO_SWO
- net TEMP_SENSOR renamed TEMP_SENS1
- new net: R17.1, U6.7 (PG10)
- no-connect marks 0 -> 16
Other:
- note removed: "OPAMP_FLR_IN"
- note removed: "OPAMP_FLR_OUT"
- moved on the sheet: C21, C22, C23, C24, C25, C26, JP5, JP6, L2, R16, SW1, Y1
