File: bldc_driver_hw/HALL_EFF_SENSOR.kicad_sch (KiCad schematic)
At the start: 6 parts

Commit message: schematic finished pcb in progress
Parts:
- renumbered C19 to C69, C20 to C70, C60 to C71, R35 to R72, R45 to R73, R46 to R74
Changed lines of the file:
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@@
 		(dnp no)
 		(fields_autoplaced yes)
-		(property "Reference" "#PWR0110"
+		(property "Reference" "#PWR0149"
 			(at 151.13 68.58 0)
 			(effects
@@
 			(project "bldc_driver_hw"
 				(path "/7f946e06-72d3-4343-93fe-84e8bb5001be/f2fa74ce-bfa7-4251-8bc0-1b2737017ea5"
-					(reference "#PWR0110")
+					(reference "#PWR0149")
 					(unit 1)
 				)
@@
 		(dnp no)
 		(fields_autoplaced yes)
-		(property "Reference" "#PWR0109"
+		(property "Reference" "#PWR0147"
 			(at 142.24 68.58 0)
 			(effects
@@
 			(project ""
 				(path "/7f946e06-72d3-4343-93fe-84e8bb5001be/f2fa74ce-bfa7-4251-8bc0-1b2737017ea5"
-					(reference "#PWR0109")
+					(reference "#PWR0147")
 					(unit 1)
 				)
@@
 		(dnp yes)
 		(fields_autoplaced yes)
-		(property "Reference" "R45"
+		(property "Reference" "R73"
 			(at 153.67 71.1199 0)
 			(effects
@@
 			(project "bldc_driver_hw"
 				(path "/7f946e06-72d3-4343-93fe-84e8bb5001be/f2fa74ce-bfa7-4251-8bc0-1b2737017ea5"
-					(reference "R45")
+					(reference "R73")
 					(unit 1)
 				)
@@
 		(dnp no)
 		(fields_autoplaced yes)
-		(property "Reference" "#PWR0112"
+		(property "Reference" "#PWR0148"
 			(at 142.24 109.22 0)
 			(effects
@@
 			(project ""
 				(path "/7f946e06-72d3-4343-93fe-84e8bb5001be/f2fa74ce-bfa7-4251-8bc0-1b2737017ea5"
-					(reference "#PWR0112")
+					(reference "#PWR0148")
 					(unit 1)
 				)
@@
 		(dnp no)
 		(fields_autoplaced yes)
-		(property "Reference" "#PWR0114"
+		(property "Reference" "#PWR0152"
 			(at 160.02 109.22 0)
 			(effects
@@
 			(project "bldc_driver_hw"
 				(path "/7f946e06-72d3-4343-93fe-84e8bb5001be/f2fa74ce-bfa7-4251-8bc0-1b2737017ea5"
-					(reference "#PWR0114")
+					(reference "#PWR0152")
 					(unit 1)
 				)
@@
 		(dnp no)
 		(fields_autoplaced yes)
-		(property "Reference" "#PWR0111"
+		(property "Reference" "#PWR0151"
 			(at 160.02 68.58 0)
 			(effects
@@
 			(project "bldc_driver_hw"
 				(path "/7f946e06-72d3-4343-93fe-84e8bb5001be/f2fa74ce-bfa7-4251-8bc0-1b2737017ea5"
-					(reference "#PWR0111")
+					(reference "#PWR0151")
 					(unit 1)
 				)
@@
 		(dnp no)
 		(fields_autoplaced yes)
-		(property "Reference" "#PWR0113"
+		(property "Reference" "#PWR0150"
 			(at 151.13 109.22 0)
 			(effects
@@
 			(project "bldc_driver_hw"
 				(path "/7f946e06-72d3-4343-93fe-84e8bb5001be/f2fa74ce-bfa7-4251-8bc0-1b2737017ea5"
-					(reference "#PWR0113")
+					(reference "#PWR0150")
 					(unit 1)
 				)
@@
 		(dnp yes)
 		(fields_autoplaced yes)
-		(property "Reference" "R35"
+		(property "Reference" "R72"
 			(at 144.78 71.1199 0)
 			(effects
@@
 			(project ""
 				(path "/7f946e06-72d3-4343-93fe-84e8bb5001be/f2fa74ce-bfa7-4251-8bc0-1b2737017ea5"
-					(reference "R35")
+					(reference "R72")
 					(unit 1)
 				)
@@
 		(dnp yes)
 		(fields_autoplaced yes)
-		(property "Reference" "R46"
+		(property "Reference" "R74"
 			(at 162.56 71.1199 0)
 			(effects
@@
 			(project "bldc_driver_hw"
 				(path "/7f946e06-72d3-4343-93fe-84e8bb5001be/f2fa74ce-bfa7-4251-8bc0-1b2737017ea5"
-					(reference "R46")
+					(reference "R74")
 					(unit 1)
 				)
@@
 		(on_board yes)
 		(dnp yes)
-		(property "Reference" "C60"
+		(property "Reference" "C71"
 			(at 161.798 97.79 0)
 			(effects
@@
 			(project "bldc_driver_hw"
 				(path "/7f946e06-72d3-4343-93fe-84e8bb5001be/f2fa74ce-bfa7-4251-8bc0-1b2737017ea5"
-					(reference "C60")
+					(reference "C71")
 					(unit 1)
 				)
@@
 		(on_board yes)
 		(dnp yes)
-		(property "Reference" "C19"
+		(property "Reference" "C69"
 			(at 144.018 97.79 0)
 			(effects
@@
 			(project ""
 				(path "/7f946e06-72d3-4343-93fe-84e8bb5001be/f2fa74ce-bfa7-4251-8bc0-1b2737017ea5"
-					(reference "C19")
+					(reference "C69")
 					(unit 1)
 				)
@@
 		(on_board yes)
 		(dnp yes)
-		(property "Reference" "C20"
+		(property "Reference" "C70"
 			(at 152.908 97.79 0)
 			(effects
@@
 			(project "bldc_driver_hw"
 				(path "/7f946e06-72d3-4343-93fe-84e8bb5001be/f2fa74ce-bfa7-4251-8bc0-1b2737017ea5"
-					(reference "C20")
-					(unit 1)
-				)
+					(reference "C70")
+					(unit 1)
+				)
