File: bldc_driver_hw/bldc_driver_hw.kicad_pcb (KiCad board)
At the start: 4 copper layers, 100 x 100 mm, 288 parts, among them J1 Conn_01x02, J10 MR60_F, J11 Conn_01x02, J2 USB_C_Receptacle_USB2.0_16P, J3 JTAG_CONN, J4 USB_C_Receptacle_USB2.0_16P, J5 Conn_01x03_Pin, J6 Conn_01x03_Pin, J7 Conn_01x03, J8 Conn_01x03_Pin, J9 Conn_01x02, Q1 IPB026N06NATMA1, Q2 IPB026N06NATMA1, Q3 IPB026N06NATMA1, Q4 IPB026N06NATMA1, Q5 IPB026N06NATMA1, Q6 IPB026N06NATMA1, SW1 SW_Push, SW2 SW_Push, SW3 SW_Push, U1 USBLC6-2SC6, U10 INA240A1D, U11 INA240A1D, U12 SN65HVD234, U13 MCP6569, U2 USBLC6-2SC6, U3 TPS54260DGQ, U4 AMS1117-3.3, U5 MCP1501-33xSN, U6 STM32G474RETx, U7 DRV8328BRUYR, U8 ESP32-C6-MINI-1, U9 INA240A1D, Y1 24MHz

Commit message: Changed one 3 phase driver to three h-bridges and changed buck converter which sink more current
Parts:
- removed C41, C45, C46, C47: 1uF, Capacitor_SMD:C_0603_1608Metric
- removed C42: 10uF, Capacitor_SMD:C_0603_1608Metric
- removed C43: 100nF, Capacitor_SMD:C_0805_2012Metric
- removed C44: 1uF, Capacitor_SMD:C_0805_2012Metric
- removed C48: 47uF, Capacitor_THT:CP_Radial_D10.0mm_P5.00mm
- removed C8: 6.8nF, Capacitor_SMD:C_0603_1608Metric_Pad1.08x0.95mm_HandSolder
- removed J11: Conn_01x02, Connector_AMASS:AMASS_XT60-F_1x02_P7.20mm_Vertical
- removed the R18 at (357.0, 93.3)
- removed R19: 100k, Resistor_SMD:R_0603_1608Metric
- removed R20, R21: R_Small, Resistor_SMD:R_0603_1608Metric
- removed R22: 10k, Resistor_SMD:R_0603_1608Metric
- removed TP15, TP16, TP17, TP18, TP19, TP20, TP21, TP22: TestPoint, TestPoint:TestPoint_Pad_D2.0mm
- removed U7: DRV8328BRUYR, bldc_driver_footprint:QFN40P400X400X80-29N-D
- added C83: 22uF, Capacitor_SMD:C_0805_2012Metric_Pad1.18x1.45mm_HandSolder, F.Cu at (351.0, 179.5)
- added C84: 10uF, Capacitor_SMD:C_0603_1608Metric_Pad1.08x0.95mm_HandSolder, F.Cu at (346.4, 165.6)
- added C85: 100nF, Capacitor_SMD:C_0603_1608Metric_Pad1.08x0.95mm_HandSolder, F.Cu at (346.4, 168.1)
- added C86: 100nF, Capacitor_SMD:C_0603_1608Metric_Pad1.08x0.95mm_HandSolder, F.Cu at (346.4, 170.6)
- added C87: 22uF, Capacitor_SMD:C_0805_2012Metric_Pad1.18x1.45mm_HandSolder, F.Cu at (351.0, 182.5)
- added C88: 10uF, Capacitor_SMD:C_0603_1608Metric_Pad1.08x0.95mm_HandSolder, F.Cu at (346.4, 173.1)
- added C89: 100nF, Capacitor_SMD:C_0603_1608Metric_Pad1.08x0.95mm_HandSolder, F.Cu at (346.4, 175.6)
- added C90: 1uF, Capacitor_SMD:C_0603_1608Metric, F.Cu at (412.3, 66.9)
- added C91: 1uF, Capacitor_SMD:C_0603_1608Metric, F.Cu at (414.0, 30.7)
- added C92: 1uF, Capacitor_SMD:C_0603_1608Metric, F.Cu at (411.4, -7.92)
- added C93: 100nF, Capacitor_SMD:C_0603_1608Metric, F.Cu at (412.0, 74.1)
- added C94: 10uF, Capacitor_SMD:C_0603_1608Metric, F.Cu at (412.0, 75.7)
- added C95: 100nF, Capacitor_SMD:C_0603_1608Metric, F.Cu at (413.7, 37.9)
- added C96: 10uF, Capacitor_SMD:C_0603_1608Metric, F.Cu at (413.7, 39.5)
- added C97: 100nF, Capacitor_SMD:C_0603_1608Metric, F.Cu at (411.0, -0.72)
- added C98: 10uF, Capacitor_SMD:C_0603_1608Metric, F.Cu at (411.0, 0.85)
- added D20: SS24, Diode_SMD:D_SMA, F.Cu at (416.3, 74.4)
- added D21: SS24, Diode_SMD:D_SMA, F.Cu at (418.0, 38.2)
- added D22: SS24, Diode_SMD:D_SMA, F.Cu at (415.4, -0.42)
- added L4: 4,7uH, bldc_driver_footprint:INDPM5452X300N, F.Cu at (352.8, 174.5)
- added R101: 10k, Resistor_SMD:R_0603_1608Metric_Pad0.98x0.95mm_HandSolder, F.Cu at (346.4, 178.1)
- added R102: 10k, Resistor_SMD:R_0603_1608Metric_Pad0.98x0.95mm_HandSolder, F.Cu at (346.4, 180.6)
- added R103: 56k, Resistor_SMD:R_0603_1608Metric_Pad0.98x0.95mm_HandSolder, F.Cu at (346.4, 183.1)
- added R104: 10k, Resistor_SMD:R_0603_1608Metric_Pad0.98x0.95mm_HandSolder, F.Cu at (346.4, 185.7)
- added R105: 10k, Resistor_SMD:R_0603_1608Metric, F.Cu at (405.9, 67.7)
- added R106: 10k, Resistor_SMD:R_0603_1608Metric, F.Cu at (407.6, 31.6)
- added R107: 10k, Resistor_SMD:R_0603_1608Metric, F.Cu at (404.9, -7.05)
- added R108: 10k, Resistor_SMD:R_0603_1608Metric, F.Cu at (405.9, 70.7)
- added R109: 10k, Resistor_SMD:R_0603_1608Metric, F.Cu at (407.6, 34.5)
- added R110: 10k, Resistor_SMD:R_0603_1608Metric, F.Cu at (404.9, -4.13)
- added TP38: TestPoint, TestPoint:TestPoint_Pad_D2.0mm, F.Cu at (355.5, 184.8)
- added U14: TPS54360DDA, Package_SO:TI_SO-PowerPAD-8_ThermalVias, F.Cu at (441.3, 153.1)
- added U15: UCC27288, Package_SO:SOIC-8_3.9x4.9mm_P1.27mm, F.Cu at (410.6, 70.5)
- added U16: UCC27288, Package_SO:SOIC-8_3.9x4.9mm_P1.27mm, F.Cu at (412.3, 34.3)
- added U17: UCC27288, Package_SO:SOIC-8_3.9x4.9mm_P1.27mm, F.Cu at (409.6, -4.33)
- C7: value 100nF -> 1.8nF
- L1: footprint Inductor_SMD:L_Vishay_IHLP-4040 -> Inductor_SMD:L_Bourns_SRP1050WA
- R12: value 100k -> 44.2k
- R13: value 680k -> 250k
- R14: value 52.3k -> 147k; footprint Resistor_SMD:R_0603_1608Metric_Pad0.98x0.95mm_HandSolder -> Resistor_SMD:R_0603_1608Metric
- R15: value 10k -> 10.5k; footprint Resistor_SMD:R_0603_1608Metric_Pad0.98x0.95mm_HandSolder -> Resistor_SMD:R_0603_1608Metric
- R18: renamed from NMT1; footprint Resistor_SMD:R_0603_1608Metric_Pad0.98x0.95mm_HandSolder -> Resistor_SMD:R_0603_1608Metric
- U3: value TPS54260DGQ -> TPS562201DDCR; footprint Package_SO:MSOP-10-1EP_3x3mm_P0.5mm_EP2.2x3.1mm_Mask1.83x1.89mm_ThermalVias -> Package_TO_SOT_SMD:SOT-23-6_Handsoldering
- moved C7 433.9 mm to (452.5, 152.5), turned to 90 degrees
- moved C6 429.1 mm to (447.5, 152.5), turned to 90 degrees
- moved R12 423.0 mm to (450.0, 153.3)
- moved R14 421.1 mm to (448.4, 155.0), turned to 180 degrees
- moved R15 418.6 mm to (446.0, 155.8), turned to -90 degrees
- moved C5 416.7 mm to (434.9, 151.6), turned to 90 degrees
- moved C16 416.1 mm to (440.1, 135.1), turned to -90 degrees
- moved C17 414.3 mm to (438.4, 135.1), turned to -90 degrees
- moved C12 413.8 mm to (436.5, 150.3), turned to 90 degrees
- moved R13 412.6 mm to (439.5, 156.9)
- moved C18 412.6 mm to (436.7, 135.1), turned to -90 degrees
- moved R18 410.0 mm to (436.5, 155.0), turned to -90 degrees
- moved L1 409.5 mm to (446.7, 138.7), turned to 90 degrees
- moved TP8 408.2 mm to (434.9, 158.5)
- moved D4 403.2 mm to (444.0, 147.8), turned to 180 degrees
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Connections:
- net /MOTOR_CTRL/H_PHASE_U/G_IN_H renamed Net-(D7-K)
- net /MOTOR_CTRL/H_PHASE_U/G_IN_L renamed Net-(D8-K)
- net /MOTOR_CTRL/H_PHASE_V/G_IN_H renamed Net-(D15-K)
- net /MOTOR_CTRL/H_PHASE_V/G_IN_L renamed Net-(D16-K)
- net /MOTOR_CTRL/H_PHASE_W/G_IN_H renamed Net-(D11-K)
- net /MOTOR_CTRL/H_PHASE_W/G_IN_L renamed Net-(D12-K)
- C12 pad 1: Net-(U3-PH) -> Net-(U14-BOOT)
- C16 pad 1: +5VD -> +12V
- C17 pad 1: +5VD -> +12V
- C18 pad 1: +5VD -> +12V
- C6 pad 1: Net-(U3-COMP) -> Net-(U14-COMP)
- L1 pad 2: +5VD -> +12V
- R11 pad 2: Net-(U3-EN) -> Net-(U14-EN)
- R12 pad 1: Net-(U3-COMP) -> Net-(U14-COMP)
- R13 pad 1: Net-(U3-RT/CLK) -> Net-(U14-RT/CLK)
- R14 pad 1: +5VD -> +12V
- R14 pad 2: Net-(U3-VSENSE) -> Net-(U14-FB)
- R15 pad 1: Net-(U3-VSENSE) -> Net-(U14-FB)
- R18 pad 1: Net-(U3-EN) -> Net-(U14-EN)
- U3 pad 1: Net-(D4-K) -> GND
- U3 pad 2: VDD -> Net-(U3-SW)
- U3 pad 3: Net-(U3-EN) -> +12V
- U3 pad 5: Net-(U3-RT/CLK) -> Net-(U3-EN)
- U3 pad 6: unconnected-(U3-PWRGD-Pad6) -> Net-(U3-VBST)
Routing:
- net +12V: track 0.00 -> 51.8 mm
- net Net-(Q6-G): track 29.0 -> 0.00 mm
- net Net-(Q2-G): track 29.0 -> 0.00 mm
- net Net-(Q5-G): track 27.4 -> 5.99 mm
- net Net-(Q1-G): track 27.4 -> 5.99 mm
- net Net-(Q4-G): track 14.5 -> 0.00 mm
- net Net-(D8-K): track 13.8 -> 0.04 mm
- net Net-(D16-K): track 13.8 -> 0.04 mm
- net Net-(D7-A): track 13.4 -> 0.00 mm
- net Net-(D15-A): track 13.4 -> 0.00 mm
- net Net-(D22-K): track 0.00 -> 9.20 mm
- net Net-(D21-K): track 0.00 -> 9.20 mm
- net Net-(D20-K): track 0.00 -> 9.20 mm
- net Net-(D4-K): track 0.00 -> 8.68 mm, vias 0 -> 2
- net Net-(Q3-G): track 13.7 -> 5.99 mm
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- added copper zone on F.Cu, net +12V
- added copper zone on F.Cu, net Net-(D11-A)
- added copper zone on F.Cu, net Net-(D11-K)
- added copper zone on F.Cu, net Net-(D12-A)
- added copper zone on F.Cu, net Net-(D12-K)
- added copper zone on F.Cu, net Net-(D15-A)
- added copper zone on F.Cu, net Net-(D15-K)
- added copper zone on F.Cu, net Net-(D16-A)
- added copper zone on F.Cu, net Net-(D16-K)
- added copper zone on F.Cu, net Net-(D4-K)
- added copper zone on F.Cu, net Net-(D7-A)
- added copper zone on F.Cu, net Net-(D7-K)
- added copper zone on F.Cu, net Net-(D8-A)
- added copper zone on F.Cu, net Net-(D8-K)
- added copper zone on F.Cu, net Net-(Q1-G)
- added copper zone on F.Cu, net Net-(Q2-G)
- added copper zone on F.Cu, net Net-(Q3-G)
- added copper zone on F.Cu, net Net-(Q4-G)
- added copper zone on F.Cu, net Net-(Q5-G)
- added copper zone on F.Cu, net Net-(Q6-G)

Commit message: Board finished to review
Parts:
- removed C1, C2: 100nF, Capacitor_SMD:C_0603_1608Metric
- removed C69, C70, C71: 1nF, Capacitor_SMD:C_0603_1608Metric
- removed J10: MR60_F, bldc_driver_footprint:MR60-F
- removed J8: Conn_01x03_Pin, Connector_PinHeader_2.54mm:PinHeader_1x03_P2.54mm_Vertical
- removed JP2, JP3, JP4: SolderJumper_2_Open, Jumper:SolderJumper-2_P1.3mm_Open_RoundedPad1.0x1.5mm
- removed R17: 47R, Resistor_SMD:R_0603_1608Metric
- removed R72, R73, R74: 10k, Resistor_SMD:R_0603_1608Metric
- removed R89: 100k, Resistor_SMD:R_0603_1608Metric
- removed TP12, TP13, TP14, TP26, TP27, TP28, TP29, TP36, TP37, TP4: TestPoint, TestPoint:TestPoint_Pad_D2.0mm
- added C100: 100nF, Capacitor_SMD:C_0603_1608Metric, F.Cu at (128.0, 34.4)
- added C41: 470uF, Capacitor_THT:CP_Radial_D16.0mm_P7.50mm, F.Cu at (138.0, 159.0)
- added C45: 47uF, Capacitor_SMD:CP_Elec_6.3x5.4, F.Cu at (154.0, 50.0)
- added C99: 100nF, Capacitor_SMD:C_0603_1608Metric, F.Cu at (109.4, 34.3)
- added G***: LOGO, bldc_driver_footprint:Haunter, F.Cu at (146.5, 144.1)
- added H1: MountingHole, MountingHole:MountingHole_3.2mm_M3, F.Cu at (203.0, 17.5)
- added H2: MountingHole, MountingHole:MountingHole_3.2mm_M3, F.Cu at (110.0, 17.5)
- added H3: MountingHole, MountingHole:MountingHole_3.2mm_M3, F.Cu at (110.0, 160.5)
- added H4: MountingHole, MountingHole:MountingHole_3.2mm_M3, F.Cu at (203.0, 160.5)
- added TP15: TestPoint, TestPoint:TestPoint_Pad_D2.0mm, F.Cu at (110.9, 121.9)
- C10, C13, C14, C49, C9: footprint Capacitor_SMD:C_0805_2012Metric_Pad1.18x1.45mm_HandSolder -> Capacitor_SMD:C_0603_1608Metric
- C11, C12, C15, C16, C17, C18, C5, C50, C6, C7, C84, C85, C86, C88, C89: footprint Capacitor_SMD:C_0603_1608Metric_Pad1.08x0.95mm_HandSolder -> Capacitor_SMD:C_0603_1608Metric
- C3, C4, C83, C87: footprint Capacitor_SMD:C_0805_2012Metric_Pad1.18x1.45mm_HandSolder -> Capacitor_SMD:C_0805_2012Metric
- C51, C52, C53, C54, C55, C56: footprint Capacitor_SMD:C_0805_2012Metric -> Capacitor_SMD:C_1206_3216Metric
- C78, C79, C80, R82, R83, R84, R85, R86, R87, R88, R90, R91, R92, R93, R94, R95, R96, R97, U13: moved to B.Cu
- C81: footprint Capacitor_SMD:C_0805_2012Metric_Pad1.18x1.45mm_HandSolder -> Capacitor_SMD:C_0603_1608Metric; moved to B.Cu
- C82: footprint Capacitor_SMD:C_0603_1608Metric_Pad1.08x0.95mm_HandSolder -> Capacitor_SMD:C_0603_1608Metric; moved to B.Cu
- R1, R2, R25, R26, R27, R28, R29, R3, R30, R31, R32, R8: footprint Capacitor_SMD:C_0603_1608Metric -> Resistor_SMD:R_0603_1608Metric
- R23, R24: footprint Resistor_SMD:R_0805_2012Metric -> Resistor_SMD:R_0603_1608Metric
- R42, R53, R64: footprint Resistor_SMD:R_0805_2012Metric -> Resistor_SMD:R_1206_3216Metric
- R43, R54, R65: value R_snub -> R_SNUB; footprint Resistor_SMD:R_0805_2012Metric -> Resistor_SMD:R_1206_3216Metric
- U8: footprint RF_Module:ESP32-C6-MINI-1 -> bldc_driver_footprint:XCVR_ESP32-C6-MINI-1-H4
- moved R13 321.7 mm to (117.9, 150.0), turned to -90 degrees
- moved R11 321.5 mm to (113.5, 146.3), turned to 0 degrees
- moved C16 320.8 mm to (119.4, 127.2)
- moved U14 320.8 mm to (120.6, 145.2)
- moved C12 320.8 mm to (115.8, 142.4)
- moved C17 320.8 mm to (117.7, 127.2)
- moved C18 320.8 mm to (116.0, 127.2)
- moved C6 320.8 mm to (126.8, 144.6)
- moved C7 320.8 mm to (131.8, 144.6)
- moved D4 320.8 mm to (123.3, 139.9)
- moved L1 320.8 mm to (126.0, 130.8)
- moved R12 320.8 mm to (129.3, 145.4)
- moved R14 320.8 mm to (127.7, 147.1)
- moved R15 320.8 mm to (125.3, 147.9)
- moved R18 320.8 mm to (115.8, 147.1)
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Connections:
- J7 pad 1: /CAN_TRANSCIEVER/CAN_H -> /CAN_TRANSCIEVER/CAN_L
- J7 pad 2: /CAN_TRANSCIEVER/CAN_L -> /CAN_TRANSCIEVER/CAN_H
- J9 pad 1: GND -> +48V
- J9 pad 2: +48V -> GND
- R84 pad 1: /BEMF_SENS/PHASE_V -> /BEMF_SENS/PHASE_W
- R86 pad 1: /BEMF_SENS/PHASE_W -> /BEMF_SENS/PHASE_V
- R92 pad 1: Net-(U13C-+) -> Net-(U13D-+)
- R94 pad 1: Net-(U13B-+) -> Net-(U13C-+)
- R95 pad 1: /BEMF_SENS/BEMF_V -> /BEMF_SENS/BEMF_W
- R95 pad 2: Net-(U13C-+) -> Net-(U13D-+)
- R97 pad 1: /BEMF_SENS/BEMF_W -> /BEMF_SENS/BEMF_V
- R97 pad 2: Net-(U13B-+) -> Net-(U13C-+)
- R98 pad 2: /BEMF_SENS/BEMF_W -> /BEMF_SENS/BEMF_V
- R99 pad 2: /BEMF_SENS/BEMF_V -> /BEMF_SENS/BEMF_W
- U13 pad 12: unconnected-(U13D-+-Pad12) -> Net-(U13D-+)
- U13 pad 13: unconnected-(U13D---Pad13) -> /BEMF_SENS/V_BEMF
- U13 pad 14: unconnected-(U13-Pad14) -> /BEMF_SENS/BEMF_W
- U13 pad 5: Net-(U13B-+) -> unconnected-(U13B-+-Pad5)
- U13 pad 6: /BEMF_SENS/V_BEMF -> unconnected-(U13B---Pad6)
- U13 pad 7: /BEMF_SENS/BEMF_W -> unconnected-(U13-Pad7)
- U6 pad 13: /MCU/TEMP_SENS2 -> /MCU/TEMP_SENS1
- U6 pad 2: /CAN_TRANSCIEVER/CAN_EN -> unconnected-(U6-PC13-Pad2)
- U6 pad 20: /MCU/ADC_CSA_V -> /MCU/ADC_CSA_U
- U6 pad 22: /MCU/ADC_CSA_U -> /MCU/ADC_CSA_V
- U6 pad 24: /MCU/TEMP_SENS1 -> /MCU/TEMP_SENS2
- U6 pad 40: /MCU/IN_H_V -> /MCU/IN_L_V
- U6 pad 41: /MCU/IN_L_V -> /MCU/IN_H_V
- U6 pad 42: /MCU/IN_H_U -> /MCU/IN_L_U
- U6 pad 43: /MCU/IN_L_U -> /MCU/IN_H_U
- U6 pad 58: unconnected-(U6-PB5-Pad58) -> /CAN_TRANSCIEVER/CAN_EN
- U6 pad 7: Net-(U6-PG10) -> /NRESET
- U8 pad 10: unconnected-(U8-IO5-Pad10) -> /RADIO/WIFI_READY
- U8 pad 15: /RADIO/CONNECTED -> unconnected-(U8-IO6-Pad15)
- U8 pad 16: /RADIO/WIFI_READY -> unconnected-(U8-IO7-Pad16)
- U8 pad 9: unconnected-(U8-IO4-Pad9) -> /RADIO/CONNECTED
Routing:
- net +3.3V: track 43.3 -> 526.2 mm, vias 0 -> 29
- net +12V: track 51.8 -> 220.3 mm, vias 0 -> 25
- net /MCU/ADC_CSA_W: track 0.00 -> 106.5 mm, vias 0 -> 2
- net /BEMF_SENS/PHASE_W: track 0.00 -> 86.5 mm, vias 0 -> 2
- net /MCU/TEMP_SENS2: track 0.00 -> 78.3 mm, vias 0 -> 4
- net GND: track 0.00 -> 75.4 mm, vias 0 -> 628
- net /MCU/ADC_CSA_V: track 0.00 -> 74.4 mm, vias 0 -> 4
- net /MCU/TEMP_SENS1: track 0.00 -> 72.1 mm, vias 0 -> 6
- net VBUS: track 0.00 -> 70.6 mm, vias 0 -> 3
- net /MCU/ADC_CSA_U: track 0.00 -> 65.0 mm, vias 0 -> 4
- net /BEMF_SENS/BEMF_V: track 0.00 -> 63.6 mm, vias 0 -> 5
- net /MCU/IN_H_U: track 2.23 -> 63.6 mm
- net /MCU/IN_L_U: track 2.23 -> 63.3 mm
- net /BEMF_SENS/BEMF_U: track 0.00 -> 60.2 mm, vias 0 -> 3
- net /BEMF_SENS/PHASE_U: track 0.00 -> 55.8 mm, vias 0 -> 2
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- added copper zone on B.Cu, net +12V
- added copper zone on B.Cu, net +3.3V
- added copper zone on F.Cu, net +3.3V
- added copper zone on B.Cu, net +48V
- added copper zone on F.Cu, net +48V
- added copper zone on F.Cu, net +5V
- added copper zone on F.Cu, net +5VD
- added copper zone on F.Cu, net /BEMF_SENS/PHASE_U
- added copper zone on F.Cu, net /BEMF_SENS/PHASE_V
- added copper zone on F.Cu, net /BEMF_SENS/PHASE_W
- added copper zone on B.Cu, net GND
- added copper zone on F.Cu, net GND
- added copper zone on B.Cu, net Net-(U3-SW)
- added copper zone on F.Cu, net Net-(U3-SW)
Other:
- board size 100 x 100 mm -> 100 x 150 mm
- copper layers 4 -> 2

Commit message: wip
Routing:
- net +3.3V: track 526.2 -> 523.6 mm
- net GND: vias 628 -> 627

Commit message: wip
Parts:
- added J10: MR60_F, bldc_driver_footprint:MR60-F, F.Cu at (252.8, 105.1)
- C78, C79, C80, C81, C82, R82, R83, R84, R85, R86, R87, R88, R90, R91, R92, R93, R94, R95, R96, R97, U13: moved to F.Cu
- moved TP25 75.6 mm to (220.7, 66.9)
- moved TP3 66.6 mm to (217.6, 61.5)
- moved TP1 65.6 mm to (215.7, 65.4)
- moved R97 21.7 mm to (154.2, 96.9), turned to 0 degrees
- moved R90 21.5 mm to (151.8, 95.3)
- moved R86 21.4 mm to (155.8, 101.6)
- moved R94 21.1 mm to (153.4, 99.2)
- moved R83 21.0 mm to (151.5, 86.1), turned to 180 degrees
- moved C78 20.9 mm to (151.5, 84.5), turned to 180 degrees
- moved R88 20.9 mm to (151.8, 90.7)
- moved R96 18.8 mm to (154.6, 87.6), turned to 0 degrees
- moved C80 18.1 mm to (155.0, 99.3), turned to 90 degrees
- moved R87 17.8 mm to (156.6, 99.2), turned to 90 degrees
- moved C81 17.6 mm to (157.9, 86.1)
- moved C82 17.5 mm to (157.9, 87.6)
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Connections:
- R84 pad 1: /BEMF_SENS/PHASE_W -> /BEMF_SENS/PHASE_V
- R86 pad 1: /BEMF_SENS/PHASE_V -> /BEMF_SENS/PHASE_W
- R93 pad 1: Net-(U13A-+) -> Net-(U13B-+)
- R95 pad 1: /BEMF_SENS/BEMF_W -> /BEMF_SENS/BEMF_V
- R96 pad 2: Net-(U13A-+) -> Net-(U13B-+)
- R97 pad 1: /BEMF_SENS/BEMF_V -> /BEMF_SENS/BEMF_W
- R98 pad 2: /BEMF_SENS/BEMF_V -> /BEMF_SENS/BEMF_W
- R99 pad 2: /BEMF_SENS/BEMF_W -> /BEMF_SENS/BEMF_V
- U13 pad 1: /BEMF_SENS/BEMF_U -> unconnected-(U13-Pad1)
- U13 pad 14: /BEMF_SENS/BEMF_W -> /BEMF_SENS/BEMF_V
- U13 pad 2: /BEMF_SENS/V_BEMF -> unconnected-(U13A---Pad2)
- U13 pad 3: Net-(U13A-+) -> unconnected-(U13A-+-Pad3)
- U13 pad 5: unconnected-(U13B-+-Pad5) -> Net-(U13B-+)
- U13 pad 6: unconnected-(U13B---Pad6) -> /BEMF_SENS/V_BEMF
- U13 pad 7: unconnected-(U13-Pad7) -> /BEMF_SENS/BEMF_U
- U13 pad 8: /BEMF_SENS/BEMF_V -> /BEMF_SENS/BEMF_W
Routing:
- net /BEMF_SENS/PHASE_V: track 36.6 -> 69.6 mm
- net /BEMF_SENS/PHASE_U: track 55.8 -> 87.9 mm, vias 2 -> 4
- net /BEMF_SENS/BEMF_U: track 60.2 -> 35.1 mm, vias 3 -> 2
- net +3.3V: track 523.6 -> 499.4 mm
- net +12V: track 220.3 -> 199.1 mm, vias 25 -> 23
- net /BEMF_SENS/PHASE_W: track 86.5 -> 71.5 mm
- net /BEMF_SENS/BEMF_V: track 63.6 -> 53.9 mm, vias 5 -> 4
- net /BEMF_SENS/BEMF_W: track 50.0 -> 40.3 mm, vias 3 -> 4
- net Net-(U13A-+): track 4.21 -> 0.00 mm
- net /MCU/IN_H_V: track 24.0 -> 28.1 mm
- net /MCU/IN_L_U: track 63.3 -> 67.3 mm
- net Net-(U13B-+): track 0.00 -> 3.96 mm
- net /MCU/IN_H_U: track 63.6 -> 67.5 mm
- net /MCU/TEMP_SENS1: track 72.1 -> 75.9 mm
- net Net-(C80-Pad1): track 6.29 -> 10.0 mm
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
Commit message: wip
Parts:
- removed J10: MR60_F, bldc_driver_footprint:MR60-F
- removed JP1: SolderJumper_2_Open, Jumper:SolderJumper-2_P1.3mm_Open_RoundedPad1.0x1.5mm
- removed TP1, TP2, TP3: TestPoint, TestPoint:TestPoint_Pad_D2.0mm
- removed U1: USBLC6-2SC6, Package_TO_SOT_SMD:SOT-23-6
- added H5: MountingHole, MountingHole:MountingHole_3.2mm_M3, F.Cu at (147.0, 116.0)
- added H6: MountingHole, MountingHole:MountingHole_3.2mm_M3, F.Cu at (163.0, 53.0)
- added U7: USBLC6-2SC6, Package_TO_SOT_SMD:SOT-23-6, F.Cu at (117.6, 47.3)
- R101, R102, R103, R104, R12, R13: footprint Resistor_SMD:R_0603_1608Metric_Pad0.98x0.95mm_HandSolder -> Resistor_SMD:R_0603_1608Metric
- moved TP25 61.0 mm to (170.5, 101.5)
- moved R10 1.88 mm to (132.6, 62.8), turned to 0 degrees
- moved U2 1.36 mm to (117.6, 58.5), turned to 0 degrees
- moved R9 0.95 mm to (130.2, 63.6)
- moved H1 0.10 mm to (203.1, 17.5)
- moved H4 0.10 mm to (203.1, 160.5)
Connections:
- J2 pad A6: /MCU/USB_D+ -> Net-(J2-D+-PadA6)
- J2 pad A7: /MCU/USB_D- -> Net-(J2-D--PadA7)
- J2 pad B6: /MCU/USB_D+ -> Net-(J2-D+-PadA6)
- J2 pad B7: /MCU/USB_D- -> Net-(J2-D--PadA7)
- J3 pad 7: Net-(J3-Pin_7) -> /MCU/JTRST
- J4 pad A6: /RADIO/D+ -> Net-(J4-D+-PadA6)
- J4 pad A7: /RADIO/D- -> Net-(J4-D--PadA7)
- J4 pad B6: /RADIO/D+ -> Net-(J4-D+-PadA6)
- J4 pad B7: /RADIO/D- -> Net-(J4-D--PadA7)
- U2 pad 1: /MCU/USB_D- -> Net-(J2-D--PadA7)
- U2 pad 3: /MCU/USB_D- -> Net-(J2-D+-PadA6)
- U2 pad 6: /MCU/USB_D+ -> /MCU/USB_D-
Routing:
- net GND: track 75.3 -> 116.9 mm, vias 547 -> 804
- net +12V: track 199.1 -> 218.5 mm, vias 23 -> 22
- net /MCU/USB_D-: track 41.0 -> 30.2 mm
- net /RADIO/D-: track 27.2 -> 17.0 mm
- net /MCU/USB_D+: track 37.9 -> 28.5 mm
- net /BEMF_SENS/BEMF_V: track 53.9 -> 62.9 mm
- net /RADIO/D+: track 27.8 -> 19.5 mm
- net Net-(J2-D--PadA7): track 0.00 -> 6.71 mm
- net Net-(J4-D--PadA7): track 0.00 -> 6.50 mm
- net Net-(J2-D+-PadA6): track 0.00 -> 5.88 mm
- net Net-(J4-D+-PadA6): track 0.00 -> 5.67 mm
- net +3.3V: track 499.4 -> 503.7 mm
- net VBUS2: track 53.1 -> 56.3 mm
- net Net-(J3-Pin_7): track 3.18 -> 0.00 mm
- net VBUS: track 70.6 -> 73.6 mm
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Other:
- outline, holes or cut-outs redrawn
- board text added: "24-60V"
- board text added: "BOOT"
- board text added: "CANH"
- board text added: "CANL"
- board text added: "Designed by Tetes & Żak"
- board text added: "GND"
- board text added: "RST"
- board text added: "RST GND TDI TRST TDO GND TCK GND TMS 3.3V"
- board text added: "RX"
- board text added: "TX"
