File: bldc_driver_hw/bldc_driver_hw.kicad_sch (KiCad schematic)
At the start: 0 parts

Commit message: wip
Parts:
- added J1: USB_C_Receptacle_USB2.0_16P, Connector_USB:USB_C_Receptacle_GCT_USB4105-xx-A_16P_TopMnt_Horizontal, symbol Connector:USB_C_Receptacle_USB2.0_16P
- added J2: Conn_01x03_Pin, Connector_PinHeader_2.54mm:PinHeader_1x03_P2.54mm_Vertical, symbol Connector:Conn_01x03_Pin
- added R3, R4: 5.1k, Capacitor_SMD:C_0603_1608Metric, symbol Device:R_Small
Connections:
- new net: J1.B5 (CC2), R3.1
- new net: J1.A5 (CC1), R4.1
- new net GND: J1.A1 (GND), J1.A12 (GND), J1.B1 (GND), J1.B12 (GND), J1.S1 (SHIELD), J2.1 (Pin_1), R3.2, R4.2
- new net RADIO/D+: J1.A6 (D+), J1.B6 (D+)
- new net RADIO/D-: J1.A7 (D-), J1.B7 (D-)
- new net RADIO/UART0_RX: J2.2 (Pin_2)
- new net RADIO/UART0_TX: J2.3 (Pin_3)
- new net VBUS: J1.A4 (VBUS), J1.A9 (VBUS), J1.B4 (VBUS), J1.B9 (VBUS)
- no-connect marks 0 -> 2
Other:
- sheet RADIO ports: added D+, D-, UART0_RX, UART0_TX, UART_MOTOR_RX, UART_MOTOR_TX; removed none

Commit message: wip
Parts:
- added C61, C62: 100nF, Capacitor_SMD:C_0603_1608Metric, symbol Device:C_Small
- added J3: USB_C_Receptacle_USB2.0_16P, Connector_USB:USB_C_Receptacle_GCT_USB4105-xx-A_16P_TopMnt_Horizontal, symbol Connector:USB_C_Receptacle_USB2.0_16P
- added J4: MR30, Connector_AMASS:AMASS_MR30PW-FB_1x03_P3.50mm_Horizontal, symbol Connector_Generic:Conn_01x03
- added J5, J6: Conn_01x03_Pin, Connector_PinHeader_2.54mm:PinHeader_1x03_P2.54mm_Vertical, symbol Connector:Conn_01x03_Pin
- added R24, R34: 5.1k, Capacitor_SMD:C_0603_1608Metric, symbol Device:R_Small
- added U10, U11: USBLC6-2SC6, Package_TO_SOT_SMD:SOT-23-6, symbol Power_Protection:USBLC6-2SC6
Connections:
- net GND: now also C61.2, C62.2, J3.A1 (GND), J3.A12 (GND), J3.B1 (GND), J3.B12 (GND), J3.S1 (SHIELD), J6.1 (Pin_1), R24.2, R34.2, U10.2 (GND), U11.2 (GND)
- net RADIO/D+: now also U11.4 (I/O2), U11.6 (I/O1)
- net RADIO/D-: now also U11.1 (I/O1), U11.3 (I/O2)
- net VBUS: now also C62.1, U11.5 (VBUS)
- new net: J3.A5 (CC1), R24.1
- new net: J3.B5 (CC2), R34.1
- new net CAN_TRANSCIEVER/CAN_H: J6.3 (Pin_3)
- new net CAN_TRANSCIEVER/CAN_L: J6.2 (Pin_2)
- new net HALL_EFF_SENSOR/HALL_IN_U: J5.3 (Pin_3)
- new net HALL_EFF_SENSOR/HALL_IN_V: J5.2 (Pin_2)
- new net HALL_EFF_SENSOR/HALL_IN_W: J5.1 (Pin_1)
- new net MCU/USB_D+: J3.A6 (D+), J3.B6 (D+), U10.4 (I/O2), U10.6 (I/O1)
- new net MCU/USB_D-: J3.A7 (D-), J3.B7 (D-), U10.1 (I/O1), U10.3 (I/O2)
- new net MOTOR_CTRL/PHASE_U: J4.1 (Pin_1)
- new net MOTOR_CTRL/PHASE_V: J4.3 (Pin_3)
- new net MOTOR_CTRL/PHASE_W: J4.2 (Pin_2)
- new net VBUS2: C61.1, J3.A4 (VBUS), J3.A9 (VBUS), J3.B4 (VBUS), J3.B9 (VBUS), U10.5 (VBUS)
- no-connect marks 2 -> 4
Other:
- added sheet BEMF_SENS (BEMF_SENS.kicad_sch)
- added sheet CAN_TRANSCIEVER (CAN_TRANSCIEVER.kicad_sch)
- added sheet HALL_EFF_SENSOR (HALL_EFF_SENSOR.kicad_sch)
- sheet MCU ports: added ADC_CSA_U, ADC_CSA_V, ADC_CSA_W, CAN_EN, CAN_RX, CAN_TX, HALL_EFF_U, HALL_EFF_V, HALL_EFF_W, IN_H_U, IN_H_V, IN_H_W, IN_L_U, IN_L_V, IN_L_W, TEMP_SENSOR, UART_MOTOR_RX, UART_MOTOR_TX, USB_D+, USB_D-; removed none
- sheet MOTOR_CTRL ports: added CURR_U, CURR_V, CURR_W, IN_H_U, IN_H_V, IN_H_W, IN_L_U, IN_L_V, IN_L_W, IRQ_FAIL, PHASE_U, PHASE_V, PHASE_W, TEMP_SENSOR; removed none
- moved on the sheet: J2

Commit message: wip
Connections:
- net MOTOR_CTRL/PHASE_U renamed BEMF_SENS/PHASE_U
- net MOTOR_CTRL/PHASE_V renamed BEMF_SENS/PHASE_V
- net MOTOR_CTRL/PHASE_W renamed BEMF_SENS/PHASE_W
Other:
- sheet BEMF_SENS ports: added BEMF_U, BEMF_V, BEMF_W, PHASE_U, PHASE_V, PHASE_W; removed none
Changed lines of the file:
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@@
 	)
 	(junction
+		(at 266.7 100.33)
+		(diameter 0)
+		(color 0 0 0 0)
+	)
+	(junction
 		(at 78.74 96.52)
 		(diameter 0)
@@
 	)
 	(junction
+		(at 262.89 97.79)
+		(diameter 0)
+		(color 0 0 0 0)
+	)
+	(junction
 		(at 48.26 41.91)
 		(diameter 0)
@@
 		(color 0 0 0 0)
 	)
+	(junction
+		(at 259.08 95.25)
+		(diameter 0)
+		(color 0 0 0 0)
+	)
 	(no_connect
 		(at 44.45 119.38)
@@
 	(wire
 		(pts
-			(xy 267.97 100.33) (xy 255.27 100.33)
+			(xy 267.97 100.33) (xy 266.7 100.33)
 		)
 		(stroke
@@
 	(wire
 		(pts
+			(xy 266.7 142.24) (xy 266.7 100.33)
+		)
+		(stroke
+			(width 0)
+			(type default)
+		)
+	)
+	(wire
+		(pts
 			(xy 46.99 96.52) (xy 44.45 96.52)
 		)
@@
 	(wire
 		(pts
+			(xy 262.89 97.79) (xy 267.97 97.79)
+		)
+		(stroke
+			(width 0)
+			(type default)
+		)
+	)
+	(wire
+		(pts
 			(xy 154.94 102.87) (xy 204.47 102.87)
 		)
@@
 	(wire
 		(pts
+			(xy 262.89 139.7) (xy 262.89 97.79)
+		)
+		(stroke
+			(width 0)
+			(type default)
+		)
+	)
+	(wire
+		(pts
 			(xy 154.94 86.36) (xy 204.47 86.36)
 		)
@@
 	(wire
 		(pts
+			(xy 259.08 95.25) (xy 267.97 95.25)
+		)
+		(stroke
+			(width 0)
+			(type default)
+		)
+	)
+	(wire
+		(pts
 			(xy 60.96 36.83) (xy 60.96 34.29)
 		)
@@
 	(wire
 		(pts
+			(xy 246.38 142.24) (xy 266.7 142.24)
+		)
+		(stroke
+			(width 0)
+			(type default)
+		)
+	)
+	(wire
+		(pts
 			(xy 82.55 40.64) (xy 82.55 41.91)
 		)
@@
 	(wire
 		(pts
-			(xy 255.27 95.25) (xy 267.97 95.25)
+			(xy 255.27 95.25) (xy 259.08 95.25)
 		)
 		(stroke
@@
 	(wire
 		(pts
+			(xy 266.7 100.33) (xy 255.27 100.33)
+		)
+		(stroke
+			(width 0)
+			(type default)
+		)
+	)
+	(wire
+		(pts
 			(xy 91.44 34.29) (xy 91.44 39.37)
 		)
@@
 	(wire
 		(pts
-			(xy 246.38 97.79) (xy 267.97 97.79)
+			(xy 246.38 97.79) (xy 262.89 97.79)
 		)
 		(stroke
@@
 	(wire
 		(pts
+			(xy 259.08 137.16) (xy 259.08 95.25)
+		)
+		(stroke
+			(width 0)
+			(type default)
+		)
+	)
+	(wire
+		(pts
 			(xy 71.12 110.49) (xy 71.12 109.22)
 		)
@@
 	(wire
 		(pts
+			(xy 246.38 139.7) (xy 262.89 139.7)
+		)
+		(stroke
+			(width 0)
+			(type default)
+		)
+	)
+	(wire
+		(pts
 			(xy 60.96 27.94) (xy 54.61 27.94)
 		)
@@
 	(wire
 		(pts
+			(xy 246.38 137.16) (xy 259.08 137.16)
+		)
+		(stroke
+			(width 0)
+			(type default)
+		)
+	)
+	(wire
+		(pts
 			(xy 191.77 31.75) (xy 198.12 31.75)
 		)
@@
 			)
 		)
+		(pin "PHASE_W" input
+			(at 246.38 139.7 0)
+			(effects
+				(font
+					(size 1.27 1.27)
+				)
+				(justify right)
+			)
+		)
+		(pin "PHASE_V" input
+			(at 246.38 142.24 0)
+			(effects
+				(font
+					(size 1.27 1.27)
+				)
+				(justify right)
+			)
+		)
+		(pin "BEMF_U" output
+			(at 215.9 137.16 180)
+			(effects
+				(font
+					(size 1.27 1.27)
+				)
+				(justify left)
+			)
+		)
+		(pin "PHASE_U" input
+			(at 246.38 137.16 0)
+			(effects
+				(font
+					(size 1.27 1.27)
+				)
+				(justify right)
+			)
+		)
+		(pin "BEMF_W" output
+			(at 215.9 139.7 180)
+			(effects
+				(font
+					(size 1.27 1.27)
+				)
+				(justify left)
+			)
+		)
+		(pin "BEMF_V" output
+			(at 215.9 142.24 180)
+			(effects
+				(font
+					(size 1.27 1.27)
+				)
+				(justify left)
+			)
+		)

Commit message: schematic finished pcb in progress
Parts:
- added J1: Conn_01x02, TerminalBlock_4Ucon:TerminalBlock_4Ucon_1x02_P3.50mm_Horizontal, symbol Connector_Generic:Conn_01x02
- added J3: JTAG_CONN, Connector_PinHeader_2.54mm:PinHeader_2x05_P2.54mm_Vertical, symbol Connector_Generic:Conn_02x05_Odd_Even
- added J7: Conn_01x03, TerminalBlock_4Ucon:TerminalBlock_4Ucon_1x03_P3.50mm_Horizontal, symbol Connector_Generic:Conn_01x03
- added J9: Conn_01x02, Connector_AMASS:AMASS_XT60-F_1x02_P7.20mm_Vertical, symbol Connector_Generic:Conn_01x02
- added JP1, JP2, JP3, JP4: SolderJumper_2_Open, Jumper:SolderJumper-2_P1.3mm_Open_RoundedPad1.0x1.5mm, symbol Jumper:SolderJumper_2_Open
- added R1, R2, R3, R8: 10k, Capacitor_SMD:C_0603_1608Metric, symbol Device:R_Small
- added R10, R9: 47R, Resistor_SMD:R_0603_1608Metric, symbol Device:R_Small
- added TP1, TP2, TP3: TestPoint, TestPoint:TestPoint_Pad_D2.0mm, symbol Connector:TestPoint
- J10: renamed from J4; value MR30 -> MR60_F; footprint Connector_AMASS:AMASS_MR30PW-FB_1x03_P3.50mm_Horizontal -> bldc_driver_footprint:MR60-F
- renumbered C62 to C1, C61 to C2, J3 to J2, J1 to J4, J2 to J5, J5 to J8, R24 to R4, R34 to R5, R4 to R6, R3 to R7, U11 to U1, U10 to U2
Connections:
- net BEMF_SENS/BEMF_U: now also JP4.1 (A), TP3.1
- net BEMF_SENS/BEMF_V: now also JP3.1 (A), TP2.1
- net BEMF_SENS/BEMF_W: now also JP2.2 (B), TP1.1
- net BEMF_SENS/PHASE_V: now also J10.2 (Pin_2); no longer J10.3 (Pin_3)
- net BEMF_SENS/PHASE_W: now also J10.3 (Pin_3); no longer J10.2 (Pin_2)
- net CAN_TRANSCIEVER/CAN_H: now also J7.1 (Pin_1); no longer J6.3 (Pin_3)
- net CAN_TRANSCIEVER/CAN_L: now also J7.2 (Pin_2); no longer J6.2 (Pin_2)
- net GND: now also J1.1 (Pin_1), J3.3 (Pin_3), J3.5 (Pin_5), J3.9 (Pin_9), J7.3 (Pin_3), J9.1 (Pin_1), R1.1
- net HALL_EFF_SENSOR/HALL_OUT_U: now also JP4.2 (B)
- net HALL_EFF_SENSOR/HALL_OUT_V: now also JP3.2 (B)
- net HALL_EFF_SENSOR/HALL_OUT_W: now also JP2.1 (A)
- new net: J3.7 (Pin_7), JP1.2 (B)
- new net +3.3V: J3.1 (Pin_1), R2.2, R3.2, R8.2
- new net +48V: J9.2 (Pin_2)
- new net JTCK_SWCLK: J3.4 (Pin_4), R1.2, R9.2
- new net JTDI: J3.8 (Pin_8), R3.1
- new net JTDO_SWO: J3.6 (Pin_6)
- new net JTMS_SWDIO: J3.2 (Pin_2), R10.2, R2.1
- new net MCU/JTCK_SWCLK: R9.1
- new net MCU/JTMS_SWDIO: R10.1
- new net MCU/JTRST: JP1.1 (A), R8.1
- new net MCU/UART5_RX: J6.3 (Pin_3)
- new net MCU/UART5_TX: J6.2 (Pin_2)
- new net NRESET: J3.10 (Pin_10)
- new net VDD: J1.2 (Pin_2)
Other:
- sheet MCU ports: added B_H_SENS_U, B_H_SENS_V, B_H_SENS_W, H_BRIDGE_IRQ, JTCK_SWCLK, JTDI, JTDO_SWO, JTMS_SWDIO, JTRST, NRESET, TEMP_SENS1, TEMP_SENS2, UART5_RX, UART5_TX; removed HALL_EFF_U, HALL_EFF_V, HALL_EFF_W, TEMP_SENSOR
- sheet MOTOR_CTRL ports: added TEMP_SENSOR1, TEMP_SENSOR2; removed TEMP_SENSOR

Commit message: Board finished to review
Parts:
- removed C1, C2: 100nF, Capacitor_SMD:C_0603_1608Metric, symbol Device:C_Small
- removed J8: Conn_01x03_Pin, Connector_PinHeader_2.54mm:PinHeader_1x03_P2.54mm_Vertical, symbol Connector:Conn_01x03_Pin
- removed JP2, JP3, JP4: SolderJumper_2_Open, Jumper:SolderJumper-2_P1.3mm_Open_RoundedPad1.0x1.5mm, symbol Jumper:SolderJumper_2_Open
- added H1, H2, H3, H4: MountingHole, MountingHole:MountingHole_3.2mm_M3, symbol Mechanical:MountingHole
- R1, R2, R3, R8: footprint Capacitor_SMD:C_0603_1608Metric -> Resistor_SMD:R_0603_1608Metric
Connections:
- net +48V: now also J9.1 (Pin_1); no longer J9.2 (Pin_2)
- net CAN_TRANSCIEVER/CAN_H: now also J7.2 (Pin_2); no longer J7.1 (Pin_1)
- net CAN_TRANSCIEVER/CAN_L: now also J7.1 (Pin_1); no longer J7.2 (Pin_2)
- net GND: now also J9.2 (Pin_2); no longer J9.1 (Pin_1)
Other:
- removed sheet HALL_EFF_SENSOR
- moved on the sheet: J9

Commit message: wip
Other:
- moved on the sheet: H1, H2, H3, H4
Changed lines of the file:
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@@
 	(symbol
 		(lib_id "Mechanical:MountingHole")
-		(at 231.14 58.42 0)
+		(at 157.48 179.07 0)
 		(unit 1)
 		(exclude_from_sim yes)
@@
 		(fields_autoplaced yes)
 		(property "Reference" "H2"
-			(at 233.68 57.1499 0)
+			(at 160.02 177.7999 0)
 			(effects
 				(font
@@
 		)
 		(property "Value" "MountingHole"
-			(at 233.68 59.6899 0)
+			(at 160.02 180.3399 0)
 			(effects
 				(font
@@
 		)
 		(property "Footprint" "MountingHole:MountingHole_3.2mm_M3"
-			(at 231.14 58.42 0)
+			(at 157.48 179.07 0)
 			(effects
 				(font
@@
 		)
 		(property "Datasheet" "~"
-			(at 231.14 58.42 0)
+			(at 157.48 179.07 0)
 			(effects
 				(font
@@
 		)
 		(property "Description" "Mounting Hole without connection"
-			(at 231.14 58.42 0)
+			(at 157.48 179.07 0)
 			(effects
 				(font
@@
 	(symbol
 		(lib_id "Mechanical:MountingHole")
-		(at 231.14 64.77 0)
+		(at 157.48 185.42 0)
 		(unit 1)
 		(exclude_from_sim yes)
@@
 		(fields_autoplaced yes)
 		(property "Reference" "H3"
-			(at 233.68 63.4999 0)
+			(at 160.02 184.1499 0)
 			(effects
 				(font
@@
 		)
 		(property "Value" "MountingHole"
-			(at 233.68 66.0399 0)
+			(at 160.02 186.6899 0)
 			(effects
 				(font
@@
 		)
 		(property "Footprint" "MountingHole:MountingHole_3.2mm_M3"
-			(at 231.14 64.77 0)
+			(at 157.48 185.42 0)
 			(effects
 				(font
@@
 		)
 		(property "Datasheet" "~"
-			(at 231.14 64.77 0)
+			(at 157.48 185.42 0)
 			(effects
 				(font
@@
 		)
 		(property "Description" "Mounting Hole without connection"
-			(at 231.14 64.77 0)
+			(at 157.48 185.42 0)
 			(effects
 				(font
@@
 	(symbol
 		(lib_id "Mechanical:MountingHole")
-		(at 231.14 52.07 0)
+		(at 157.48 172.72 0)
 		(unit 1)
 		(exclude_from_sim yes)
@@
 		(fields_autoplaced yes)
 		(property "Reference" "H1"
-			(at 233.68 50.7999 0)
+			(at 160.02 171.4499 0)
 			(effects
 				(font
@@
 		)
 		(property "Value" "MountingHole"
-			(at 233.68 53.3399 0)
+			(at 160.02 173.9899 0)
 			(effects
 				(font
@@
 		)
 		(property "Footprint" "MountingHole:MountingHole_3.2mm_M3"
-			(at 231.14 52.07 0)
+			(at 157.48 172.72 0)
 			(effects
 				(font
@@
 		)
 		(property "Datasheet" "~"
-			(at 231.14 52.07 0)
+			(at 157.48 172.72 0)
 			(effects
 				(font
@@
 		)
 		(property "Description" "Mounting Hole without connection"
-			(at 231.14 52.07 0)
+			(at 157.48 172.72 0)
 			(effects
 				(font
@@
 	(symbol
 		(lib_id "Mechanical:MountingHole")
-		(at 231.1169 70.2908 0)
+		(at 157.4569 190.9408 0)
 		(unit 1)
 		(exclude_from_sim yes)
@@
 		(fields_autoplaced yes)
 		(property "Reference" "H4"
-			(at 233.6569 69.0207 0)
+			(at 159.9969 189.6707 0)
 			(effects
 				(font
@@
 		)
 		(property "Value" "MountingHole"
-			(at 233.6569 71.5607 0)
+			(at 159.9969 192.2107 0)
 			(effects
 				(font
@@
 		)
 		(property "Footprint" "MountingHole:MountingHole_3.2mm_M3"
-			(at 231.1169 70.2908 0)
+			(at 157.4569 190.9408 0)
 			(effects
 				(font
@@
 		)
 		(property "Datasheet" "~"
-			(at 231.1169 70.2908 0)
+			(at 157.4569 190.9408 0)
 			(effects
 				(font
@@
 		)
 		(property "Description" "Mounting Hole without connection"
-			(at 231.1169 70.2908 0)
+			(at 157.4569 190.9408 0)
 			(effects
 				(font

Commit message: wip
Parts:
- removed JP1: SolderJumper_2_Open, Jumper:SolderJumper-2_P1.3mm_Open_RoundedPad1.0x1.5mm, symbol Jumper:SolderJumper_2_Open
- removed TP1, TP2, TP3: TestPoint, TestPoint:TestPoint_Pad_D2.0mm, symbol Connector:TestPoint
- removed U1: USBLC6-2SC6, Package_TO_SOT_SMD:SOT-23-6, symbol Power_Protection:USBLC6-2SC6
- added H5, H6: MountingHole, MountingHole:MountingHole_3.2mm_M3, symbol Mechanical:MountingHole
- added U7: USBLC6-2SC6, Package_TO_SOT_SMD:SOT-23-6, symbol Power_Protection:USBLC6-2SC6
Connections:
- net GND: now also U7.2 (GND)
- net MCU/JTRST: now also J3.7 (Pin_7)
- net MCU/USB_D+: no longer J2.A6 (D+), J2.B6 (D+), U2.6 (I/O1)
- net MCU/USB_D-: now also U2.6 (I/O1); no longer J2.A7 (D-), J2.B7 (D-), U2.1 (I/O1), U2.3 (I/O2)
- net RADIO/D+: now also U7.4 (I/O2); no longer J4.A6 (D+), J4.B6 (D+)
- net RADIO/D-: now also U7.6 (I/O1); no longer J4.A7 (D-), J4.B7 (D-)
- net VBUS: now also U7.5 (VBUS)
- new net: J2.A7 (D-), J2.B7 (D-), U2.1 (I/O1)
- new net: J2.A6 (D+), J2.B6 (D+), U2.3 (I/O2)
- new net: J4.A7 (D-), J4.B7 (D-), U7.1 (I/O1)
- new net: J4.A6 (D+), J4.B6 (D+), U7.3 (I/O2)
Other:
- note added: "TO_DO DOPASOWAC IMPEDANCYJNIE USB -> ( NIE WIEM CZY JEST SENS ALE MOZNA SIE NAUCZYC_ SPRAWDZIC BOOT0"
- moved on the sheet: U2

Commit message: board finished
Parts:
- added JP1: SolderJumper_2_Open, Jumper:SolderJumper-2_P1.3mm_Open_Pad1.0x1.5mm, symbol Jumper:SolderJumper_2_Open
Connections:
- net +48V: now also JP1.1 (A)
- net VDD: now also JP1.2 (B)
Other:
- note removed: "TO_DO DOPASOWAC IMPEDANCYJNIE USB -> ( NIE WIEM CZY JEST SENS ALE MOZNA SIE NAUCZYC_ SPRAWDZIC BOOT0"
- moved on the sheet: J9
