File: bldc_driver_hw/BEMF_SENS.kicad_sch (KiCad schematic)
At the start: 24 parts, among them U13 MCP6569

Commit message: finished_board
Parts:
- R92, R93, R94: value R_Small -> 0R; LCSC (none) -> C15402
- R95, R96, R97: value R_Small -> 510k; LCSC (none) -> C23192

Commit message: finished
Parts:
- C78, C79, C80: now fitted; now left out of the parts list
- R92, R93, R94: LCSC C15402 -> C21189
- U13: now left out of the parts list
Changed lines of the file:
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@@
 			)
 		)
-		(property "LCSC" "C15402"
+		(property "LCSC" "C21189"
 			(at 120.65 114.3 0)
 			(effects
@@
 		(unit 5)
 		(exclude_from_sim no)
-		(in_bom yes)
+		(in_bom no)
 		(on_board yes)
 		(dnp no)
@@
 		(unit 1)
 		(exclude_from_sim no)
-		(in_bom yes)
-		(on_board yes)
-		(dnp yes)
+		(in_bom no)
+		(on_board yes)
+		(dnp no)
 		(fields_autoplaced yes)
 		(property "Reference" "C80"
@@
 		(unit 1)
 		(exclude_from_sim no)
-		(in_bom yes)
-		(on_board yes)
-		(dnp yes)
+		(in_bom no)
+		(on_board yes)
+		(dnp no)
 		(fields_autoplaced yes)
 		(property "Reference" "C79"
@@
 		(unit 1)
 		(exclude_from_sim no)
-		(in_bom yes)
-		(on_board yes)
-		(dnp yes)
+		(in_bom no)
+		(on_board yes)
+		(dnp no)
 		(fields_autoplaced yes)
 		(property "Reference" "C78"
@@
 		(unit 4)
 		(exclude_from_sim no)
-		(in_bom yes)
+		(in_bom no)
 		(on_board yes)
 		(dnp no)
@@
 			)
 		)
-		(property "LCSC" "C15402"
+		(property "LCSC" "C21189"
 			(at 123.19 81.28 0)
 			(effects
@@
 		(unit 2)
 		(exclude_from_sim no)
-		(in_bom yes)
+		(in_bom no)
 		(on_board yes)
 		(dnp no)
@@
 		(unit 3)
 		(exclude_from_sim no)
-		(in_bom yes)
+		(in_bom no)
 		(on_board yes)
 		(dnp no)
@@
 		(unit 1)
 		(exclude_from_sim no)
-		(in_bom yes)
+		(in_bom no)
 		(on_board yes)
 		(dnp no)
@@
 			)
 		)
-		(property "LCSC" "C15402"
+		(property "LCSC" "C21189"
 			(at 123.19 49.53 0)
 			(effects
